Commit message: feature/noetic

File: prostbot_description/robots/create_circles_asus_xtion_pro.urdf.xacro (robot description, xacro)
@@ -10,6 +10,6 @@
   <xacro:include filename="$(find prostbot_description)/urdf/stacks/circles.urdf.xacro"/>
   <xacro:include filename="$(find prostbot_description)/urdf/sensors/asus_xtion_pro.urdf.xacro"/>
-  <create/>
-  <stack_circles parent="base_link"/>
-  <sensor_asus_xtion_pro  parent="base_link"/>
+  <xacro:create/>
+  <xacro:stack_circles parent="base_link"/>
+  <xacro:sensor_asus_xtion_pro  parent="base_link"/>
 </robot>

File: prostbot_description/robots/kobuki_hexagons_astra.urdf.xacro (robot description, xacro)
@@ -7,5 +7,5 @@
 <robot name="turtlebot" xmlns:xacro="http://ros.org/wiki/xacro">
   <xacro:include filename="$(find prostbot_description)/urdf/turtlebot_common_library.urdf.xacro" />
-  <xacro:include filename="$(find base_description)/urdf/kobuki.urdf.xacro" />
+  <xacro:include filename="$(find base_description)/urdf/base.urdf.xacro" />
   <xacro:include filename="$(find prostbot_description)/urdf/stacks/hexagons.urdf.xacro"/>
   <xacro:include filename="$(find prostbot_description)/urdf/sensors/astra.urdf.xacro"/>

File: prostbot_description/robots/kobuki_hexagons_asus_xtion_pro.urdf.xacro (robot description, xacro)
@@ -7,5 +7,5 @@
 <robot name="turtlebot" xmlns:xacro="http://ros.org/wiki/xacro">
   <xacro:include filename="$(find prostbot_description)/urdf/turtlebot_common_library.urdf.xacro" />
-  <xacro:include filename="$(find base_description)/urdf/kobuki.urdf.xacro" />
+  <xacro:include filename="$(find base_description)/urdf/base.urdf.xacro" />
   <xacro:include filename="$(find prostbot_description)/urdf/stacks/hexagons.urdf.xacro"/>
   <xacro:include filename="$(find prostbot_description)/urdf/sensors/asus_xtion_pro.urdf.xacro"/>

File: prostbot_description/robots/kobuki_hexagons_kinect.urdf.xacro (robot description, xacro)
@@ -7,5 +7,5 @@
 <robot name="turtlebot" xmlns:xacro="http://ros.org/wiki/xacro">
   <xacro:include filename="$(find prostbot_description)/urdf/turtlebot_common_library.urdf.xacro" />
-  <xacro:include filename="$(find base_description)/urdf/kobuki.urdf.xacro" />
+  <xacro:include filename="$(find base_description)/urdf/base.urdf.xacro" />
   <xacro:include filename="$(find prostbot_description)/urdf/stacks/hexagons.urdf.xacro"/>
   <xacro:include filename="$(find prostbot_description)/urdf/sensors/kinect.urdf.xacro"/>

File: prostbot_description/robots/kobuki_hexagons_r200.urdf.xacro (robot description, xacro)
@@ -7,5 +7,5 @@
 <robot name="turtlebot" xmlns:xacro="http://ros.org/wiki/xacro">
   <xacro:include filename="$(find prostbot_description)/urdf/turtlebot_common_library.urdf.xacro" />
-  <xacro:include filename="$(find base_description)/urdf/kobuki.urdf.xacro" />
+  <xacro:include filename="$(find base_description)/urdf/base.urdf.xacro" />
   <xacro:include filename="$(find prostbot_description)/urdf/stacks/hexagons.urdf.xacro"/>
   <xacro:include filename="$(find prostbot_description)/urdf/sensors/r200.urdf.xacro"/>

File: prostbot_description/urdf/sensors/asus_xtion_pro_offset.urdf.xacro (robot description, xacro)
@@ -9,5 +9,5 @@
   <xacro:property name="asus_xtion_pro_offset_cam_rel_rgb_py"   value="-0.0220" />
   <!-- Parameterised in part by the values in turtlebot_properties.urdf.xacro -->
-  <xacro:macro name="sensor_asus_xtion_pro_offset" params="parent">
+  <xacro:macro name="sensor_asus_xtion_pro_offset" params="parent asus_xtion_pro_offset_cam_py}">
     <joint name="camera_rgb_joint" type="fixed">
       <origin xyz="${cam_px} ${asus_xtion_pro_offset_cam_py} ${cam_pz}"
@@ -64,4 +64,31 @@
     <!-- RGBD sensor for simulation, same as Kinect -->
     <turtlebot_sim_3dsensor/>
+    <!-- Asus mount -->
+    <joint name="mount_xtion_pro_joint" type="fixed">
+      <origin xyz="-0.1024 0.0 0.272" rpy="0 0 0"/>
+      <parent link="${parent}"/>
+      <child link="mount_xtion_pro_link"/>
+    </joint>
+    <link name="mount_xtion_pro_link">
+      <visual>
+        <origin xyz="0 0 0" rpy="${-M_PI/2} 0 0"/>
+        <geometry>
+          <mesh filename="package://prostbot_description/meshes/sensors/xtion_pro_stack.dae"/>
+        </geometry>
+      </visual>
+      <collision>
+        <origin xyz="0.0 0.0 0.0" rpy="0 0 0" />
+        <geometry>
+        <box size="0.0330 0.2760 0.0120"/>
+      </geometry>
+      </collision>
+      <inertial>
+        <mass value="0.170" />
+        <origin xyz="0 0 0" />
+        <inertia ixx="0.001152600" ixy="0.0" ixz="0.0"
+                 iyy="0.000148934" iyz="0.0"
+                 izz="0.001154654" />
+      </inertial>
+    </link>
   </xacro:macro>
 </robot>

File: turtlebot2/turtlebot/turtlebot_description/robots/roomba_circles_kinect.urdf.xacro (robot description, xacro)
@@ -6,8 +6,8 @@
 -->
 <robot name="turtlebot" xmlns:xacro="http://ros.org/wiki/xacro">
-  <xacro:include filename="$(find turtlebot_description)/urdf/turtlebot_common_library.urdf.xacro" />
+  <xacro:include filename="$(find prostbot_description)/urdf/turtlebot_common_library.urdf.xacro" />
   <xacro:include filename="$(find create_description)/urdf/create.urdf.xacro"/>
-  <xacro:include filename="$(find turtlebot_description)/urdf/stacks/circles.urdf.xacro"/>
-  <xacro:include filename="$(find turtlebot_description)/urdf/sensors/kinect.urdf.xacro"/>
+  <xacro:include filename="$(find prostbot_description)/urdf/stacks/circles.urdf.xacro"/>
+  <xacro:include filename="$(find prostbot_description)/urdf/sensors/kinect.urdf.xacro"/>
   <xacro:create/>
   <xacro:stack_circles parent="base_link"/>

Commit message: add

File: prostbot_description/robots/create_circles_asus_xtion_pro.urdf.xacro (robot description, xacro)
@@ -10,6 +10,6 @@
   <xacro:include filename="$(find prostbot_description)/urdf/stacks/circles.urdf.xacro"/>
   <xacro:include filename="$(find prostbot_description)/urdf/sensors/asus_xtion_pro.urdf.xacro"/>
-  <xacro:create/>
-  <xacro:stack_circles parent="base_link"/>
-  <xacro:sensor_asus_xtion_pro  parent="base_link"/>
+  <create/>
+  <stack_circles parent="base_link"/>
+  <sensor_asus_xtion_pro  parent="base_link"/>
 </robot>

File: prostbot_description/robots/kobuki_hexagons_astra.urdf.xacro (robot description, xacro)
@@ -7,5 +7,5 @@
 <robot name="turtlebot" xmlns:xacro="http://ros.org/wiki/xacro">
   <xacro:include filename="$(find prostbot_description)/urdf/turtlebot_common_library.urdf.xacro" />
-  <xacro:include filename="$(find base_description)/urdf/base.urdf.xacro" />
+  <xacro:include filename="$(find base_description)/urdf/kobuki.urdf.xacro" />
   <xacro:include filename="$(find prostbot_description)/urdf/stacks/hexagons.urdf.xacro"/>
   <xacro:include filename="$(find prostbot_description)/urdf/sensors/astra.urdf.xacro"/>

File: prostbot_description/robots/kobuki_hexagons_asus_xtion_pro.urdf.xacro (robot description, xacro)
@@ -7,5 +7,5 @@
 <robot name="turtlebot" xmlns:xacro="http://ros.org/wiki/xacro">
   <xacro:include filename="$(find prostbot_description)/urdf/turtlebot_common_library.urdf.xacro" />
-  <xacro:include filename="$(find base_description)/urdf/base.urdf.xacro" />
+  <xacro:include filename="$(find base_description)/urdf/kobuki.urdf.xacro" />
   <xacro:include filename="$(find prostbot_description)/urdf/stacks/hexagons.urdf.xacro"/>
   <xacro:include filename="$(find prostbot_description)/urdf/sensors/asus_xtion_pro.urdf.xacro"/>

File: prostbot_description/robots/kobuki_hexagons_kinect.urdf.xacro (robot description, xacro)
@@ -7,5 +7,5 @@
 <robot name="turtlebot" xmlns:xacro="http://ros.org/wiki/xacro">
   <xacro:include filename="$(find prostbot_description)/urdf/turtlebot_common_library.urdf.xacro" />
-  <xacro:include filename="$(find base_description)/urdf/base.urdf.xacro" />
+  <xacro:include filename="$(find base_description)/urdf/kobuki.urdf.xacro" />
   <xacro:include filename="$(find prostbot_description)/urdf/stacks/hexagons.urdf.xacro"/>
   <xacro:include filename="$(find prostbot_description)/urdf/sensors/kinect.urdf.xacro"/>

File: prostbot_description/robots/kobuki_hexagons_r200.urdf.xacro (robot description, xacro)
@@ -7,5 +7,5 @@
 <robot name="turtlebot" xmlns:xacro="http://ros.org/wiki/xacro">
   <xacro:include filename="$(find prostbot_description)/urdf/turtlebot_common_library.urdf.xacro" />
-  <xacro:include filename="$(find base_description)/urdf/base.urdf.xacro" />
+  <xacro:include filename="$(find base_description)/urdf/kobuki.urdf.xacro" />
   <xacro:include filename="$(find prostbot_description)/urdf/stacks/hexagons.urdf.xacro"/>
   <xacro:include filename="$(find prostbot_description)/urdf/sensors/r200.urdf.xacro"/>

File: prostbot_description/urdf/sensors/asus_xtion_pro_offset.urdf.xacro (robot description, xacro)
@@ -9,5 +9,5 @@
   <xacro:property name="asus_xtion_pro_offset_cam_rel_rgb_py"   value="-0.0220" />
   <!-- Parameterised in part by the values in turtlebot_properties.urdf.xacro -->
-  <xacro:macro name="sensor_asus_xtion_pro_offset" params="parent asus_xtion_pro_offset_cam_py}">
+  <xacro:macro name="sensor_asus_xtion_pro_offset" params="parent">
     <joint name="camera_rgb_joint" type="fixed">
       <origin xyz="${cam_px} ${asus_xtion_pro_offset_cam_py} ${cam_pz}"
@@ -64,31 +64,4 @@
     <!-- RGBD sensor for simulation, same as Kinect -->
     <turtlebot_sim_3dsensor/>
-    <!-- Asus mount -->
-    <joint name="mount_xtion_pro_joint" type="fixed">
-      <origin xyz="-0.1024 0.0 0.272" rpy="0 0 0"/>
-      <parent link="${parent}"/>
-      <child link="mount_xtion_pro_link"/>
-    </joint>
-    <link name="mount_xtion_pro_link">
-      <visual>
-        <origin xyz="0 0 0" rpy="${-M_PI/2} 0 0"/>
-        <geometry>
-          <mesh filename="package://prostbot_description/meshes/sensors/xtion_pro_stack.dae"/>
-        </geometry>
-      </visual>
-      <collision>
-        <origin xyz="0.0 0.0 0.0" rpy="0 0 0" />
-        <geometry>
-        <box size="0.0330 0.2760 0.0120"/>
-      </geometry>
-      </collision>
-      <inertial>
-        <mass value="0.170" />
-        <origin xyz="0 0 0" />
-        <inertia ixx="0.001152600" ixy="0.0" ixz="0.0"
-                 iyy="0.000148934" iyz="0.0"
-                 izz="0.001154654" />
-      </inertial>
-    </link>
   </xacro:macro>
 </robot>
