Commit message: updated for simulator

File: prostbot_description/urdf/kobuki_gazebo.urdf.xacro (robot description, xacro)
@@ -161,20 +161,20 @@
 	  </gazebo>
 	  <gazebo>
-	    <plugin name="kobuki_controller" filename="libgazebo_ros_kobuki.so">
-	      <publish_tf>1</publish_tf>
-	      <left_wheel_joint_name>wheel_left_joint</left_wheel_joint_name>
-	      <right_wheel_joint_name>wheel_right_joint</right_wheel_joint_name>
-	      <wheel_separation>.230</wheel_separation>
-	      <wheel_diameter>0.070</wheel_diameter>
-	      <torque>1.0</torque>
-	      <velocity_command_timeout>0.6</velocity_command_timeout>
-	      <cliff_sensor_left_name>cliff_sensor_left</cliff_sensor_left_name>
-	      <cliff_sensor_center_name>cliff_sensor_front</cliff_sensor_center_name>
-	      <cliff_sensor_right_name>cliff_sensor_right</cliff_sensor_right_name>
-	      <cliff_detection_threshold>0.04</cliff_detection_threshold>
-	      <bumper_name>bumpers</bumper_name>
+      <plugin name="kobuki_controller" filename="libgazebo_ros_kobuki.so">
+        <publish_tf>1</publish_tf>
+        <left_wheel_joint_name>wheel_l_joint</left_wheel_joint_name>
+        <right_wheel_joint_name>wheel_r_joint</right_wheel_joint_name>
+        <wheel_separation>.230</wheel_separation>
+        <wheel_diameter>0.070</wheel_diameter>
+        <torque>1.0</torque>
+        <velocity_command_timeout>0.6</velocity_command_timeout>
+        <cliff_sensor_left_name>cliff_sensor_left</cliff_sensor_left_name>
+        <cliff_sensor_center_name>cliff_sensor_front</cliff_sensor_center_name>
+        <cliff_sensor_right_name>cliff_sensor_right</cliff_sensor_right_name>
+        <cliff_detection_threshold>0.04</cliff_detection_threshold>
+        <bumper_name>bumpers</bumper_name>
         <imu_name>imu</imu_name>
-	    </plugin>
-	  </gazebo>
+      </plugin>
+    </gazebo>
     <!-- camera -->
     <gazebo reference="cam_link">

File: prostbot_description/urdf/sensors/asus_xtion_pro_offset.urdf.xacro (robot description, xacro)
@@ -9,5 +9,5 @@
   <xacro:property name="asus_xtion_pro_offset_cam_rel_rgb_py"   value="-0.0220" />
   <!-- Parameterised in part by the values in turtlebot_properties.urdf.xacro -->
-  <xacro:macro name="sensor_asus_xtion_pro_offset" params="parent asus_xtion_pro_offset_cam_py}">
+  <xacro:macro name="sensor_asus_xtion_pro_offset" params="parent">
     <joint name="camera_rgb_joint" type="fixed">
       <origin xyz="${cam_px} ${asus_xtion_pro_offset_cam_py} ${cam_pz}"
@@ -63,32 +63,5 @@
     <link name="camera_depth_optical_frame"/>
     <!-- RGBD sensor for simulation, same as Kinect -->
-    <turtlebot_sim_3dsensor/>
-    <!-- Asus mount -->
-    <joint name="mount_xtion_pro_joint" type="fixed">
-      <origin xyz="-0.1024 0.0 0.272" rpy="0 0 0"/>
-      <parent link="${parent}"/>
-      <child link="mount_xtion_pro_link"/>
-    </joint>
-    <link name="mount_xtion_pro_link">
-      <visual>
-        <origin xyz="0 0 0" rpy="${-M_PI/2} 0 0"/>
-        <geometry>
-          <mesh filename="package://prostbot_description/meshes/sensors/xtion_pro_stack.dae"/>
-        </geometry>
-      </visual>
-      <collision>
-        <origin xyz="0.0 0.0 0.0" rpy="0 0 0" />
-        <geometry>
-        <box size="0.0330 0.2760 0.0120"/>
-      </geometry>
-      </collision>
-      <inertial>
-        <mass value="0.170" />
-        <origin xyz="0 0 0" />
-        <inertia ixx="0.001152600" ixy="0.0" ixz="0.0"
-                 iyy="0.000148934" iyz="0.0"
-                 izz="0.001154654" />
-      </inertial>
-    </link>
+    <xacro:turtlebot_sim_3dsensor/>
   </xacro:macro>
 </robot>

File: prostbot_description/urdf/stacks/hexagons.urdf.xacro (robot description, xacro)
@@ -127,10 +127,10 @@
   -->
   <xacro:macro name="stack_hexagons" params="parent">
-    <stack_bottom_pole parent="${parent}" number="0" x_loc= "0.120" y_loc= "0.082" z_loc="0.1028"/>
-    <stack_bottom_pole parent="${parent}" number="1" x_loc= "0.055" y_loc= "0.120" z_loc="0.1028"/>
-    <stack_bottom_pole parent="${parent}" number="2" x_loc="-0.055" y_loc= "0.120" z_loc="0.1028"/>
-    <stack_bottom_pole parent="${parent}" number="3" x_loc= "0.120" y_loc="-0.082" z_loc="0.1028"/>
-    <stack_bottom_pole parent="${parent}" number="4" x_loc= "0.055" y_loc="-0.120" z_loc="0.1028"/>
-    <stack_bottom_pole parent="${parent}" number="5" x_loc="-0.055" y_loc="-0.120" z_loc="0.1028"/>
+    <xacro:stack_bottom_pole parent="${parent}" number="0" x_loc= "0.120" y_loc= "0.082" z_loc="0.1028"/>
+    <xacro:stack_bottom_pole parent="${parent}" number="1" x_loc= "0.055" y_loc= "0.120" z_loc="0.1028"/>
+    <xacro:stack_bottom_pole parent="${parent}" number="2" x_loc="-0.055" y_loc= "0.120" z_loc="0.1028"/>
+    <xacro:stack_bottom_pole parent="${parent}" number="3" x_loc= "0.120" y_loc="-0.082" z_loc="0.1028"/>
+    <xacro:stack_bottom_pole parent="${parent}" number="4" x_loc= "0.055" y_loc="-0.120" z_loc="0.1028"/>
+    <xacro:stack_bottom_pole parent="${parent}" number="5" x_loc="-0.055" y_loc="-0.120" z_loc="0.1028"/>
     <joint name="plate_bottom_joint" type="fixed">
       <origin xyz="0.02364 0.0 0.1306" rpy="0 0 0"/>
@@ -159,8 +159,8 @@
       </inertial>
     </link>
-    <stack_middle_pole parent="${parent}" number="0" x_loc= "0.0381" y_loc= "0.1505" z_loc="0.1640"/>
-    <stack_middle_pole parent="${parent}" number="1" x_loc= "0.0381" y_loc="-0.1505" z_loc="0.1640"/>
-    <stack_middle_pole parent="${parent}" number="2" x_loc="-0.0381" y_loc= "0.1505" z_loc="0.1640"/>
-    <stack_middle_pole parent="${parent}" number="3" x_loc="-0.0381" y_loc="-0.1505" z_loc="0.1640"/>
+    <xacro:stack_middle_pole parent="${parent}" number="0" x_loc= "0.0381" y_loc= "0.1505" z_loc="0.1640"/>
+    <xacro:stack_middle_pole parent="${parent}" number="1" x_loc= "0.0381" y_loc="-0.1505" z_loc="0.1640"/>
+    <xacro:stack_middle_pole parent="${parent}" number="2" x_loc="-0.0381" y_loc= "0.1505" z_loc="0.1640"/>
+    <xacro:stack_middle_pole parent="${parent}" number="3" x_loc="-0.0381" y_loc="-0.1505" z_loc="0.1640"/>
     <joint name="plate_middle_joint" type="fixed">
       <origin xyz="-0.01364 0.0 0.1874" rpy="0 0 0"/>
@@ -189,10 +189,10 @@
       </inertial>
     </link>
-    <stack_top_pole parent="${parent}" number="0" x_loc= "0.0381" y_loc= "0.1505" z_loc="0.2920"/>
-    <stack_top_pole parent="${parent}" number="1" x_loc= "0.0381" y_loc="-0.1505" z_loc="0.2920"/>
-    <stack_top_pole parent="${parent}" number="2" x_loc="-0.0381" y_loc= "0.1505" z_loc="0.2920"/>
-    <stack_top_pole parent="${parent}" number="3" x_loc="-0.0381" y_loc="-0.1505" z_loc="0.2920"/>
-    <stack_3d_sensor_pole parent="${parent}" number="0" x_loc="-0.1024" y_loc= "0.098" z_loc="0.2372"/>
-    <stack_3d_sensor_pole parent="${parent}" number="1" x_loc="-0.1024" y_loc="-0.098" z_loc="0.2372"/>
+    <xacro:stack_top_pole parent="${parent}" number="0" x_loc= "0.0381" y_loc= "0.1505" z_loc="0.2920"/>
+    <xacro:stack_top_pole parent="${parent}" number="1" x_loc= "0.0381" y_loc="-0.1505" z_loc="0.2920"/>
+    <xacro:stack_top_pole parent="${parent}" number="2" x_loc="-0.0381" y_loc= "0.1505" z_loc="0.2920"/>
+    <xacro:stack_top_pole parent="${parent}" number="3" x_loc="-0.0381" y_loc="-0.1505" z_loc="0.2920"/>
+    <!-- <xacro:stack_3d_sensor_pole parent="${parent}" number="0" x_loc="-0.1024" y_loc= "0.098" z_loc="0.2372"/> -->
+    <!-- <xacro:stack_3d_sensor_pole parent="${parent}" number="1" x_loc="-0.1024" y_loc="-0.098" z_loc="0.2372"/> -->
     <joint name="plate_top_joint" type="fixed">
       <origin xyz="-0.01364 0.0  0.3966" rpy="0 0 0"/>
